Commit message: Nexus Description
archivo urdf para el nexus robot

File: src/robot_description/nexus_mecanum/urdf/nexusSergio.urdf (robot description, URDF)
Before this commit: robot nexus, 16 links, 15 joints
Links:
- link base_link: geometry collision mesh filename=package://nexus_mecanum/meshes/BaseSuperior (Meshed).STL scale=0.001 0.001 0.001; visual mesh filename=package://nexus_mecanum/meshes/BaseInferior (Meshed).stl scale=0.001 0.001 0.001
